Commit message: working 2-cell miura pattern

File: miura-ori_pattern-2cells.urdf (robot description, URDF)
Before this commit: robot miura-ori_pattern, 10 links, 9 joints
Links:
- removed link base_link
- removed link wheel1
- removed link wheel1_b
- removed link wheel2
- removed link wheel2_b
- removed link wheel3
- removed link wheel3_b
- removed link wheel4
- removed link wheel4_b
- added link base_link_a, mass 0.100; collision mesh filename=mori-design-2.stl scale=1.00 1.00 1.00; visual mesh filename=mori-design-2.stl scale=1.00 1.00 1.00
- added link wheel_1_a; collision mesh filename=wheel.stl scale=1.00 1.00 1.00; visual mesh filename=wheel.stl scale=1.00 1.00 1.00
- added link wheel_1_b; collision mesh filename=wheel.stl scale=1.00 1.00 1.00; visual mesh filename=wheel.stl scale=1.00 1.00 1.00
- added link wheel_2_a; collision mesh filename=wheel.stl scale=1.00 1.00 1.00; visual mesh filename=wheel.stl scale=1.00 1.00 1.00
- added link wheel_2_b; collision mesh filename=wheel.stl scale=1.00 1.00 1.00; visual mesh filename=wheel.stl scale=1.00 1.00 1.00
- added link wheel_3_a; collision mesh filename=wheel.stl scale=1.00 1.00 1.00; visual mesh filename=wheel.stl scale=1.00 1.00 1.00
- added link wheel_3_b; collision mesh filename=wheel.stl scale=1.00 1.00 1.00; visual mesh filename=wheel.stl scale=1.00 1.00 1.00
- added link wheel_4_a; collision mesh filename=wheel.stl scale=1.00 1.00 1.00; visual mesh filename=wheel.stl scale=1.00 1.00 1.00
- added link wheel_4_b; collision mesh filename=wheel.stl scale=1.00 1.00 1.00; visual mesh filename=wheel.stl scale=1.00 1.00 1.00
Joints:
- removed joint base_link_b_joint
- removed joint joint1
- removed joint joint1_b
- removed joint joint2
- removed joint joint2_b
- removed joint joint3
- removed joint joint3_b
- removed joint joint4
- removed joint joint4_b
- added joint shaft_1_a: type continuous, parent base_link_a, child wheel_1_a, origin xyz=0.0 105.0 0 rpy=0 0 0, axis 0 1 0
- added joint shaft_1_b: type continuous, parent base_link_b, child wheel_1_b, origin xyz=-90.9326674 54.5 0 rpy=0 0 1.0472, axis 0 1 0
- added joint shaft_2_a: type continuous, parent base_link_a, child wheel_2_a, origin xyz=38.9711 22.5 0 rpy=0 0 -1.0472, axis 0 1 0
- added joint shaft_2_b: type continuous, parent base_link_b, child wheel_2_b, origin xyz=0.0 47.0 0 rpy=0 0 0.0, axis 0 1 0
- added joint shaft_3_a: type continuous, parent base_link_a, child wheel_3_a, origin xyz=129.9038 120.0 0 rpy=0 0 0, axis 0 1 0
- added joint shaft_3_b: type continuous, parent base_link_b, child wheel_3_b, origin xyz=-38.9711 174.5 0 rpy=0 0 1.0472, axis 0 1 0
- added joint shaft_4_a: type continuous, parent base_link_a, child wheel_4_a, origin xyz=90.9327 202.5 0 rpy=0 0 -1.0472, axis 0 1 0
- added joint shaft_4_b: type continuous, parent base_link_b, child wheel_4_b, origin xyz=-129.9038 182.0 0 rpy=0 0 0.0, axis 0 1 0
- added joint shaft_a_b: type revolute, parent base_link_a, child base_link_b, origin xyz=0.0 -2.0 0.0 rpy=0 0 0, axis 0 1 0, limit lower=-3.14 upper=3.14 effort=40 velocity=0.1
