Commit message: add parallelograms 3 and 4

File: miura-ori_pattern.urdf (robot description, URDF)
Before this commit: robot miura-ori_pattern, 10 links, 9 joints
Links:
- added link base_link_c; collision mesh filename=mori-design-2.stl scale=1.00 1.00 1.00; visual mesh filename=mori-design-2.stl scale=1.00 1.00 1.00
- added link base_link_d; collision mesh filename=mori-design-2.stl scale=1.00 1.00 1.00; visual mesh filename=mori-design-2.stl scale=1.00 1.00 1.00
- added link wheel1_c; collision mesh filename=wheel.stl scale=1.00 1.00 1.00; visual mesh filename=wheel.stl scale=1.00 1.00 1.00
- added link wheel1_d; collision mesh filename=wheel.stl scale=1.00 1.00 1.00; visual mesh filename=wheel.stl scale=1.00 1.00 1.00
- added link wheel2_c; collision mesh filename=wheel.stl scale=1.00 1.00 1.00; visual mesh filename=wheel.stl scale=1.00 1.00 1.00
- added link wheel2_d; collision mesh filename=wheel.stl scale=1.00 1.00 1.00; visual mesh filename=wheel.stl scale=1.00 1.00 1.00
- added link wheel3_c; collision mesh filename=wheel.stl scale=1.00 1.00 1.00; visual mesh filename=wheel.stl scale=1.00 1.00 1.00
- added link wheel3_d; collision mesh filename=wheel.stl scale=1.00 1.00 1.00; visual mesh filename=wheel.stl scale=1.00 1.00 1.00
- added link wheel4_c; collision mesh filename=wheel.stl scale=1.00 1.00 1.00; visual mesh filename=wheel.stl scale=1.00 1.00 1.00
- added link wheel4_d; collision mesh filename=wheel.stl scale=1.00 1.00 1.00; visual mesh filename=wheel.stl scale=1.00 1.00 1.00
Joints:
- added joint base_link_c_joint: type continuous, parent base_link, child base_link_c, origin xyz=0 -150 0 rpy=0 0 0, axis 0 1 0
- added joint base_link_d_joint: type continuous, parent base_link_c, child base_link_d, origin xyz=139 230 0 rpy=0 0 -2.0944, axis 0 1 0
- added joint joint1_c: type continuous, parent base_link_c, child wheel1_c, origin xyz=5 103 8 rpy=0 0 0, axis 0 1 0
- added joint joint1_d: type continuous, parent base_link_d, child wheel1_d, origin xyz=5 103 8 rpy=0 0 0, axis 0 1 0
- added joint joint2_c: type continuous, parent base_link_c, child wheel2_c, origin xyz=135 118 8 rpy=0 0 0, axis 0 1 0
- added joint joint2_d: type continuous, parent base_link_d, child wheel2_d, origin xyz=135 118 8 rpy=0 0 0, axis 0 1 0
- added joint joint3_c: type continuous, parent base_link_c, child wheel3_c, origin xyz=46 25 8 rpy=0 0 2.0944, axis 0 1 0
- added joint joint3_d: type continuous, parent base_link_d, child wheel3_d, origin xyz=46 25 8 rpy=0 0 2.0944, axis 0 1 0
- added joint joint4_c: type continuous, parent base_link_c, child wheel4_c, origin xyz=99 202 8 rpy=0 0 2.0944, axis 0 1 0
- added joint joint4_d: type continuous, parent base_link_d, child wheel4_d, origin xyz=99 202 8 rpy=0 0 2.0944, axis 0 1 0
- joint base_link_b_joint: origin xyz=140 230 0 rpy=0 0 -2.0944 -> xyz=139 230 0 rpy=0 0 -2.0944

Commit message: fix urdf prelim - not finished

File: miura-ori_pattern.urdf (robot description, URDF)
Before this commit: robot miura-ori_pattern, 20 links, 19 joints
Links:
- link base_link: mass None -> 0.100
- link base_link_b: mass None -> 0.100
- link base_link_c: mass None -> 0.100
- link base_link_d: mass None -> 0.100
Joints:
- joint base_link_b_joint: limit (none) -> lower=-3.14 upper=3.14 effort=40 velocity=0.1; type continuous -> revolute
- joint base_link_c_joint: limit (none) -> lower=-3.14 upper=3.14 effort=40 velocity=0.1; type continuous -> revolute
- joint base_link_d_joint: limit (none) -> lower=-3.14 upper=3.14 effort=40 velocity=0.1; type continuous -> revolute
- joint joint1: limit (none) -> lower=-3.14 upper=3.14 effort=40 velocity=0.1; type continuous -> revolute
- joint joint1_b: limit (none) -> lower=-3.14 upper=3.14 effort=40 velocity=0.1; type continuous -> revolute
- joint joint1_c: limit (none) -> lower=-3.14 upper=3.14 effort=40 velocity=0.1; type continuous -> revolute
- joint joint1_d: limit (none) -> lower=-3.14 upper=3.14 effort=40 velocity=0.1; type continuous -> revolute
- joint joint2: limit (none) -> lower=-3.14 upper=3.14 effort=40 velocity=0.1; type continuous -> revolute
- joint joint2_b: limit (none) -> lower=-3.14 upper=3.14 effort=40 velocity=0.1; type continuous -> revolute
- joint joint2_c: limit (none) -> lower=-3.14 upper=3.14 effort=40 velocity=0.1; type continuous -> revolute
- joint joint2_d: limit (none) -> lower=-3.14 upper=3.14 effort=40 velocity=0.1; type continuous -> revolute
- joint joint3: limit (none) -> lower=-3.14 upper=3.14 effort=40 velocity=0.1; type continuous -> revolute
- joint joint3_b: limit (none) -> lower=-3.14 upper=3.14 effort=40 velocity=0.1; type continuous -> revolute
- joint joint3_c: limit (none) -> lower=-3.14 upper=3.14 effort=40 velocity=0.1; type continuous -> revolute
- joint joint3_d: limit (none) -> lower=-3.14 upper=3.14 effort=40 velocity=0.1; type continuous -> revolute
- joint joint4: limit (none) -> lower=-3.14 upper=3.14 effort=40 velocity=0.1; type continuous -> revolute
- joint joint4_b: limit (none) -> lower=-3.14 upper=3.14 effort=40 velocity=0.1; type continuous -> revolute
- joint joint4_c: limit (none) -> lower=-3.14 upper=3.14 effort=40 velocity=0.1; type continuous -> revolute
- joint joint4_d: limit (none) -> lower=-3.14 upper=3.14 effort=40 velocity=0.1; type continuous -> revolute

Commit message: working on adding constraint to miura pattern for the last joint

File: miura-ori_pattern.urdf (robot description, URDF)
Before this commit: robot miura-ori_pattern, 20 links, 19 joints
Links:
- removed link base_link
- removed link wheel1
- removed link wheel1_b
- removed link wheel1_c
- removed link wheel1_d
- removed link wheel2
- removed link wheel2_b
- removed link wheel2_c
- removed link wheel2_d
- removed link wheel3
- removed link wheel3_b
- removed link wheel3_c
- removed link wheel3_d
- removed link wheel4
- removed link wheel4_b
- removed link wheel4_c
- removed link wheel4_d
- added link base_link_a, mass 1.420; collision mesh filename=mori-design-2.stl scale=1.00 1.00 1.00; visual mesh filename=mori-design-2.stl scale=1.00 1.00 1.00
- added link cylinder_a, mass 0.003; collision cylinder length=0.3 radius=0.03; visual cylinder length=80 radius=1.5
- added link cylinder_d, mass 0.003; collision cylinder length=0.3 radius=0.03; visual cylinder length=80 radius=1.5
- added link wheel_1_a; collision mesh filename=wheel.stl scale=1.00 1.00 1.00; visual mesh filename=wheel.stl scale=1.00 1.00 1.00
- added link wheel_1_b; collision mesh filename=wheel.stl scale=1.00 1.00 1.00; visual mesh filename=wheel.stl scale=1.00 1.00 1.00
- added link wheel_1_c; collision mesh filename=wheel.stl scale=1.00 1.00 1.00; visual mesh filename=wheel.stl scale=1.00 1.00 1.00
- added link wheel_2_a; collision mesh filename=wheel.stl scale=1.00 1.00 1.00; visual mesh filename=wheel.stl scale=1.00 1.00 1.00
- added link wheel_2_b; collision mesh filename=wheel.stl scale=1.00 1.00 1.00; visual mesh filename=wheel.stl scale=1.00 1.00 1.00
- added link wheel_2_c; collision mesh filename=wheel.stl scale=1.00 1.00 1.00; visual mesh filename=wheel.stl scale=1.00 1.00 1.00
- added link wheel_3_a; collision mesh filename=wheel.stl scale=1.00 1.00 1.00; visual mesh filename=wheel.stl scale=1.00 1.00 1.00
- added link wheel_3_b; collision mesh filename=wheel.stl scale=1.00 1.00 1.00; visual mesh filename=wheel.stl scale=1.00 1.00 1.00
- added link wheel_3_c; collision mesh filename=wheel.stl scale=1.00 1.00 1.00; visual mesh filename=wheel.stl scale=1.00 1.00 1.00
- added link wheel_4_a; collision mesh filename=wheel.stl scale=1.00 1.00 1.00; visual mesh filename=wheel.stl scale=1.00 1.00 1.00
- added link wheel_4_b; collision mesh filename=wheel.stl scale=1.00 1.00 1.00; visual mesh filename=wheel.stl scale=1.00 1.00 1.00
- added link wheel_4_c; collision mesh filename=wheel.stl scale=1.00 1.00 1.00; visual mesh filename=wheel.stl scale=1.00 1.00 1.00
- link base_link_b: mass 0.100 -> 1.420
- link base_link_c: mass 0.100 -> 1.420
- link base_link_d: mass 0.100 -> 1.420
Joints:
- removed joint base_link_b_joint
- removed joint base_link_c_joint
- removed joint base_link_d_joint
- removed joint joint1
- removed joint joint1_b
- removed joint joint1_c
- removed joint joint1_d
- removed joint joint2
- removed joint joint2_b
- removed joint joint2_c
- removed joint joint2_d
- removed joint joint3
- removed joint joint3_b
- removed joint joint3_c
- removed joint joint3_d
- removed joint joint4
- removed joint joint4_b
- removed joint joint4_c
- removed joint joint4_d
- added joint shaft_1_a: type continuous, parent base_link_a, child wheel_1_a, origin xyz=0.0 105.0 0 rpy=0 0 0, axis 0 1 0
- added joint shaft_1_b: type continuous, parent base_link_b, child wheel_1_b, origin xyz=-90.9326674 54.5 0 rpy=0 0 1.0472, axis 0 1 0
- added joint shaft_1_c: type continuous, parent base_link_c, child wheel_1_c, origin xyz=0.0 -99.0 0 rpy=0 0 0.0, axis 0 1 0
- added joint shaft_2_a: type continuous, parent base_link_a, child wheel_2_a, origin xyz=38.9711 22.5 0 rpy=0 0 -1.0472, axis 0 1 0
- added joint shaft_2_b: type continuous, parent base_link_b, child wheel_2_b, origin xyz=0.0 47.0 0 rpy=0 0 0.0, axis 0 1 0
- added joint shaft_2_c: type continuous, parent base_link_c, child wheel_2_c, origin xyz=-38.9711 -16.5 0 rpy=0 0 -1.0472, axis 0 1 0
- added joint shaft_3_a: type continuous, parent base_link_a, child wheel_3_a, origin xyz=129.9038 120.0 0 rpy=0 0 0, axis 0 1 0
- added joint shaft_3_b: type continuous, parent base_link_b, child wheel_3_b, origin xyz=-38.9711 174.5 0 rpy=0 0 1.0472, axis 0 1 0
- added joint shaft_3_c: type continuous, parent base_link_c, child wheel_3_c, origin xyz=-129.9038 -114.0 0 rpy=0 0 0.0, axis 0 1 0
- added joint shaft_4_a: type continuous, parent base_link_a, child wheel_4_a, origin xyz=90.9327 202.5 0 rpy=0 0 -1.0472, axis 0 1 0
- added joint shaft_4_b: type continuous, parent base_link_b, child wheel_4_b, origin xyz=-129.9038 182.0 0 rpy=0 0 0.0, axis 0 1 0
- added joint shaft_4_c: type continuous, parent base_link_c, child wheel_4_c, origin xyz=-90.9327 -196.5 0 rpy=0 0 -1.0472, axis 0 1 0
- added joint shaft_a_b: type revolute, parent base_link_a, child base_link_b, origin xyz=0.0 -2.0 0.0 rpy=0 0 0, axis 0 1 0, limit lower=-3.14 upper=3.14 effort=1 velocity=0.1
- added joint shaft_a_cylinder: type revolute, parent base_link_a, child cylinder_a, origin xyz=0 0 0 rpy=0 0 -1.0472, axis 0 1 0, limit lower=-3.14 upper=3.14 effort=1 velocity=0.1
- added joint shaft_b_c: type revolute, parent base_link_b, child base_link_c, origin xyz=-124.9038 74.5.0 0.0 rpy=0 0 1.0472, axis 0 1 0, limit lower=-3.14 upper=3.14 effort=1 velocity=0.1
- added joint shaft_c_d: type revolute, parent base_link_c, child base_link_d, origin xyz=-130 -219 0.0 rpy=0 0 -1.0472, axis 0 1 0, limit lower=-3.14 upper=3.14 effort=1 velocity=0.1
- added joint shaft_d_cylinder: type revolute, parent base_link_d, child cylinder_d, origin xyz=0 150 0 rpy=0 0 -1.0472, axis 0 1 0, limit lower=-3.14 upper=3.14 effort=1 velocity=0.1

Commit message: working miura pattern

File: miura-ori_pattern.urdf (robot description, URDF)
Before this commit: robot miura-ori_pattern, 18 links, 17 joints
Links:
- added link wheel_1_d; collision mesh filename=wheel.stl scale=1.00 1.00 1.00; visual mesh filename=wheel.stl scale=1.00 1.00 1.00
- added link wheel_2_d; collision mesh filename=wheel.stl scale=1.00 1.00 1.00; visual mesh filename=wheel.stl scale=1.00 1.00 1.00
- added link wheel_3_d; collision mesh filename=wheel.stl scale=1.00 1.00 1.00; visual mesh filename=wheel.stl scale=1.00 1.00 1.00
- added link wheel_4_d; collision mesh filename=wheel.stl scale=1.00 1.00 1.00; visual mesh filename=wheel.stl scale=1.00 1.00 1.00
Joints:
- added joint shaft_1_d: type continuous, parent base_link_d, child wheel_1_d, origin xyz=0.0 105.0 0 rpy=0 0 0.0, axis 0 1 0
- added joint shaft_2_d: type continuous, parent base_link_d, child wheel_2_d, origin xyz=38.9711 22.5 0 rpy=0 0 -1.0472, axis 0 1 0
- added joint shaft_3_d: type continuous, parent base_link_d, child wheel_3_d, origin xyz=129.9038 120.0 0 rpy=0 0 0, axis 0 1 0
- added joint shaft_4_d: type continuous, parent base_link_d, child wheel_4_d, origin xyz=90.9327 202.5 0 rpy=0 0 -1.0472, axis 0 1 0
- joint shaft_a_b: limit lower=-3.14 upper=3.14 effort=1 velocity=0.1 -> lower=-3.14 upper=3.14 effort=0.1 velocity=0.1
- joint shaft_a_cylinder: limit lower=-3.14 upper=3.14 effort=1 velocity=0.1 -> lower=-3.14 upper=3.14 effort=0.01 velocity=0.1
- joint shaft_b_c: limit lower=-3.14 upper=3.14 effort=1 velocity=0.1 -> (none); type revolute -> continuous
- joint shaft_c_d: limit lower=-3.14 upper=3.14 effort=1 velocity=0.1 -> lower=-3.14 upper=3.14 effort=0.1 velocity=0.1
- joint shaft_d_cylinder: limit lower=-3.14 upper=3.14 effort=1 velocity=0.1 -> lower=-3.14 upper=3.14 effort=0.01 velocity=0.1

Commit message: motor inertial updates

File: miura-ori_pattern.urdf (robot description, URDF)
Before this commit: robot miura-ori_pattern, 20 links, 19 joints
Links:
- link base_link: geometry collision mesh filename=mori-design-2.stl scale=0.10 0.10 0.10; visual mesh filename=mori-design-2.stl scale=0.10 0.10 0.10
- link base_link_b: geometry collision mesh filename=ri-design-2.stl scale=1.00 1.00 1.00; visual mesh filename=mori-design-2.stl scale=1.00 1.00 1.00
- link wheel1: geometry collision mesh filename=wheel.stl scale=0.10 0.10 0.10; visual mesh filename=wheel.stl scale=0.10 0.10 0.10
- link wheel2: geometry collision mesh filename=wheel.stl scale=0.10 0.10 0.10; visual mesh filename=wheel.stl scale=0.10 0.10 0.10
- link wheel3: geometry collision mesh filename=wheel.stl scale=0.10 0.10 0.10; visual mesh filename=wheel.stl scale=0.10 0.10 0.10
- link wheel4: geometry collision mesh filename=wheel.stl scale=0.10 0.10 0.10; visual mesh filename=wheel.stl scale=0.10 0.10 0.10

File: miura_bot_old.urdf (robot description, URDF)
Before this commit: robot miura_bot, 9 links, 8 joints
Links:
- removed link wheel_1
- removed link wheel_2
- removed link wheel_3
- removed link wheel_4
- added link wheel1; collision mesh filename=wheel.stl scale=1.00 1.00 1.00; visual mesh filename=wheel.stl scale=1.00 1.00 1.00
- added link wheel2; collision mesh filename=wheel.stl scale=1.00 1.00 1.00; visual mesh filename=wheel.stl scale=1.00 1.00 1.00
- added link wheel3; collision mesh filename=wheel.stl scale=1.00 1.00 1.00; visual mesh filename=wheel.stl scale=1.00 1.00 1.00
- added link wheel4; collision mesh filename=wheel.stl scale=1.00 1.00 1.00; visual mesh filename=wheel.stl scale=1.00 1.00 1.00
- link base_link: mass 0.100 -> None
Joints:
- removed joint shaft_1
- removed joint shaft_2
- removed joint shaft_3
- removed joint shaft_4
- added joint joint1: type continuous, parent base_link, child wheel1, origin xyz=5 103 8 rpy=0 0 0, axis 0 1 0
- added joint joint2: type continuous, parent base_link, child wheel2, origin xyz=135 118 8 rpy=0 0 0, axis 0 1 0
- added joint joint3: type continuous, parent base_link, child wheel3, origin xyz=46 25 8 rpy=0 0 2.0944, axis 0 1 0
- added joint joint4: type continuous, parent base_link, child wheel4, origin xyz=99 202 8 rpy=0 0 2.0944, axis 0 1 0
- joint jointmotor1: origin xyz=-42.9519 2.5 0 rpy=0 0 4.71238898038 -> xyz=28.0000052838 115 5 rpy=0 0 4.71238898038
- joint jointmotor2: origin xyz=42.928097162 -2.5 0 rpy=0 0 1.57079632679 -> xyz=113.9 110 5 rpy=0 0 1.57079632679
- joint jointmotor3: origin xyz=-45.641 -75.9474 0 rpy=0 0 0.523598775598 -> xyz=25.31 36.5526 5 rpy=0 0 0.523598775598
- joint jointmotor4: origin xyz=45.641 75.9474 0 rpy=0 0 3.66519142919 -> xyz=116.593 188.447 5 rpy=0 0 3.66519142919
