Commit message: updated urdf

File: miura_bot.urdf (robot description, URDF)
Before this commit: robot miura-bot, 1 links, 0 joints
Links:
- added link wheel1; collision mesh filename=C:/Users/bamlab/Desktop/liza/miura_bot/urdf/wheel.stl scale=0.01 0.01 0.01; visual mesh filename=C:/Users/bamlab/Desktop/liza/miura_bot/urdf/wheel.stl scale=0.01 0.01 0.01
- added link wheel2; collision mesh filename=C:/Users/bamlab/Desktop/liza/miura_bot/urdf/wheel.stl scale=0.01 0.01 0.01; visual mesh filename=C:/Users/bamlab/Desktop/liza/miura_bot/urdf/wheel.stl
- link base_link: geometry collision mesh filename=C:/Users/bamlab/Desktop/liza/miura_bot/urdf/mori-design-2.s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 scale=0.01 0.01 0.01; visual mesh filename=C:/Users/bamlab/Desktop/liza/miura_bot/urdf/mori-design-2.s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 scale=0.01 0.01 0.01
Joints:
- added joint joint1: type revolute, parent base_link, child wheel1, origin xyz=129.904 75 5 rpy=0 0 0, axis 0 1 0, limit lower=-1.571 upper=1.571 effort=1000.0 velocity=0.5
- added joint joint2: type revolute, parent base_link, child wheel2, origin xyz=0 150 5 rpy=0 0 0, axis 0.866 0.5 0, limit lower=-1.571 upper=1.571 effort=1000.0 velocity=0.5

Commit message: edit urdf to have proper scaling to show all links (temp: fixed joints)

File: miura_bot.urdf (robot description, URDF)
Before this commit: robot miura_bot, 3 links, 2 joints
Links:
- link base_link: geometry collision mesh filename=mori-design-2.stl scale=0.01 0.01 0.01; visual mesh filename=mori-design-2.stl scale=0.01 0.01 0.01
- link wheel1: geometry collision mesh filename=wheel.stl scale=0.01 0.01 0.01; visual mesh filename=wheel.stl scale=0.01 0.01 0.01
- link wheel2: geometry collision mesh filename=wheel.stl scale=0.01 0.01 0.01; visual mesh filename=wheel.stl scale=0.01 0.01 0.01
Joints:
- joint joint1: origin xyz=129.904 75 5 rpy=0 0 0 -> xyz=1.29904 0.75 0.05 rpy=0 0 0; type revolute -> fixed
- joint joint2: origin xyz=0 150 5 rpy=0 0 0 -> xyz=0.00 15.0 0.05 rpy=0 0 0; type revolute -> fixed

Commit message: moving miura bot (need to fix wheel origin)

File: miura_bot.urdf (robot description, URDF)
Before this commit: robot miura_bot, 3 links, 2 joints
Links:
- added link wheel3; collision mesh filename=wheel.stl scale=1.00 1.00 1.00; visual mesh filename=wheel.stl scale=1.00 1.00 1.00
- added link wheel4; collision mesh filename=wheel.stl scale=1.00 1.00 1.00; visual mesh filename=wheel.stl scale=1.00 1.00 1.00
- link base_link: geometry collision mesh filename=mori-design-2.stl scale=1.00 1.00 1.00; visual mesh filename=mori-design-2.stl scale=1.00 1.00 1.00
- link wheel1: geometry collision mesh filename=wheel.stl scale=1.00 1.00 1.00; visual mesh filename=wheel.stl scale=1.00 1.00 1.00
- link wheel2: geometry collision mesh filename=wheel.stl scale=1.00 1.00 1.00; visual mesh filename=wheel.stl scale=1.00 1.00 1.00
Joints:
- added joint joint3: type continuous, parent base_link, child wheel3, origin xyz=52 17 0 rpy=0 0 2.0944, axis 0 1 0
- added joint joint4: type continuous, parent base_link, child wheel4, origin xyz=105 196 0 rpy=0 0 2.0944, axis 0 1 0
- joint joint1: limit lower=-1.571 upper=1.571 effort=1000.0 velocity=0.5 -> (none); origin xyz=1.29904 0.75 0.05 rpy=0 0 0 -> xyz=0 103 0 rpy=0 0 0; type fixed -> continuous
- joint joint2: axis 0.866 0.5 0 -> 0 1 0; limit lower=-1.571 upper=1.571 effort=1000.0 velocity=0.5 -> (none); origin xyz=0.00 15.0 0.05 rpy=0 0 0 -> xyz=130 118 0 rpy=0 0 0; type fixed -> continuous

Commit message: fix wheel (and motor) offset from joint spinning in urdf files

File: miura_bot.urdf (robot description, URDF)
Before this commit: robot miura_bot, 5 links, 4 joints
Joints:
- joint joint1: origin xyz=0 103 0 rpy=0 0 0 -> xyz=5 103 8 rpy=0 0 0
- joint joint2: origin xyz=130 118 0 rpy=0 0 0 -> xyz=135 118 8 rpy=0 0 0
- joint joint3: origin xyz=52 17 0 rpy=0 0 2.0944 -> xyz=46 25 8 rpy=0 0 2.0944
- joint joint4: origin xyz=105 196 0 rpy=0 0 2.0944 -> xyz=99 202 8 rpy=0 0 2.0944

File: wheel_with_motor.urdf (robot description, URDF)
Before this commit: robot wheel_with_motor, 2 links, 1 joints
Joints:
- joint joint1: axis (none) -> 0 1 0; origin xyz=0 0 0 rpy=0.0 0 1.5708 -> xyz=0 0 0 rpy=0.0 0 0

Commit message: working new model of single unit cell of miura bot

File: miura_bot.urdf (robot description, URDF)
Before this commit: robot miura_bot, 5 links, 4 joints
Links:
- removed link wheel1
- removed link wheel2
- removed link wheel3
- removed link wheel4
- added link wheel_1; collision mesh filename=wheel.stl scale=1.00 1.00 1.00; visual mesh filename=wheel.stl scale=1.00 1.00 1.00
- added link wheel_2; collision mesh filename=wheel.stl scale=1.00 1.00 1.00; visual mesh filename=wheel.stl scale=1.00 1.00 1.00
- added link wheel_3; collision mesh filename=wheel.stl scale=1.00 1.00 1.00; visual mesh filename=wheel.stl scale=1.00 1.00 1.00
- added link wheel_4; collision mesh filename=wheel.stl scale=1.00 1.00 1.00; visual mesh filename=wheel.stl scale=1.00 1.00 1.00
- link base_link: mass None -> 0.100
Joints:
- removed joint joint1
- removed joint joint2
- removed joint joint3
- removed joint joint4
- added joint shaft_1: type continuous, parent base_link, child wheel_1, origin xyz=-64.9519 -7.5 0 rpy=0 0 0, axis 0 1 0
- added joint shaft_2: type continuous, parent base_link, child wheel_2, origin xyz=-25.9808 -90.0 0 rpy=0 0 -1.0472, axis 0 1 0
- added joint shaft_3: type continuous, parent base_link, child wheel_3, origin xyz=64.9519 7.5 0 rpy=0 0 0, axis 0 1 0
- added joint shaft_4: type continuous, parent base_link, child wheel_4, origin xyz=25.9808 90.0 0 rpy=0 0 -1.0472, axis 0 1 0

Commit message: added the motors as links to the urdf

File: miura_bot.urdf (robot description, URDF)
Before this commit: robot miura_bot, 5 links, 4 joints
Links:
- added link motor1; collision mesh filename=motor.stl scale=1.00 1.00 1.00; visual mesh filename=motor.stl scale=1.00 1.00 1.00
- added link motor2; collision mesh filename=motor_tip.stl scale=1.00 1.00 1.00; visual mesh filename=motor_tip.stl scale=1.00 1.00 1.00
- added link motor3; collision mesh filename=motor.stl scale=1.00 1.00 1.00; visual mesh filename=motor.stl scale=1.00 1.00 1.00
- added link motor4; collision mesh filename=motor.stl scale=1.00 1.00 1.00; visual mesh filename=motor.stl scale=1.00 1.00 1.00
Joints:
- added joint jointmotor1: type fixed, parent base_link, child motor1, origin xyz=28.0000052838 115 5 rpy=0 0 4.71238898038
- added joint jointmotor2: type fixed, parent base_link, child motor2, origin xyz=113.9 110 5 rpy=0 0 1.57079632679
- added joint jointmotor3: type fixed, parent base_link, child motor3, origin xyz=25.31 36.5526 5 rpy=0 0 0.523598775598
- added joint jointmotor4: type fixed, parent base_link, child motor4, origin xyz=116.593 188.447 5 rpy=0 0 3.66519142919

Commit message: remove motor tip

File: miura_bot.urdf (robot description, URDF)
Before this commit: robot miura_bot, 9 links, 8 joints
Links:
- link motor2: geometry collision mesh filename=motor.stl scale=1.00 1.00 1.00; visual mesh filename=motor.stl scale=1.00 1.00 1.00

Commit message: adjusted the wheel/motor positions to the flipped stl

File: miura_bot.urdf (robot description, URDF)
Before this commit: robot miura_bot, 9 links, 8 joints
Joints:
- joint jointmotor1: origin xyz=-42.9519 2.5 0 rpy=0 0 4.71238898038 -> xyz=-42.9519 -2.5 0 rpy=0 0 -4.71238898038
- joint jointmotor2: origin xyz=42.928097162 -2.5 0 rpy=0 0 1.57079632679 -> xyz=42.928097162 2.5 0 rpy=0 0 -1.57079632679
- joint jointmotor3: origin xyz=-45.641 -75.9474 0 rpy=0 0 0.523598775598 -> xyz=45.641 -75.9474 0 rpy=0 0 2.61799387799
- joint jointmotor4: origin xyz=45.641 75.9474 0 rpy=0 0 3.66519142919 -> xyz=-45.641 75.9474 0 rpy=0 0 -0.5235987756
- joint shaft_1: origin xyz=-64.9519 -7.5 0 rpy=0 0 0 -> xyz=-64.9519 7.5 0 rpy=0 0 0
- joint shaft_2: origin xyz=-25.9808 -90.0 0 rpy=0 0 -1.0472 -> xyz=25.9808 -90.0 0 rpy=0 0 1.0472
- joint shaft_3: origin xyz=64.9519 7.5 0 rpy=0 0 0 -> xyz=64.9519 -7.5 0 rpy=0 0 0
- joint shaft_4: origin xyz=25.9808 90.0 0 rpy=0 0 -1.0472 -> xyz=-25.9808 90.0 0 rpy=0 0 1.0472
